File: hardware/nrfmicro.kicad_sch (KiCad schematic)
At the start: 24 parts, among them J1 USB-C USB 2.0 MC-372, J2 Conn_01x04, J3 Conn_01x02, J4 Conn_01x04, Q1 AO3407, Q2 AO3407, U1 E73-2G4M08S1C, U2 AP2112K-3.3, U3 TP4054, U4 ProMicro, X1 32768kHz

Commit message: /** add pin */
Parts:
- removed D2: BLUE, LED_SMD:LED_0603_1608Metric, symbol Device:LED
- removed JP1: SolderJumper_2_Open, nrfmicro:Jumper_SMD, symbol Jumper:SolderJumper_2_Open
- removed R4, R8: 1K, Resistor_SMD:R_0603_1608Metric, symbol nrfmicro-rescue:R
- added J5: Conn_01x04, nrfmicro:connector_gpio_1, symbol Connector_Generic:Conn_01x04
- added J6: Conn_01x04, nrfmicro:connector_gpio_2, symbol Connector_Generic:Conn_01x04
- added R8: 1K, Resistor_SMD:R_0603_1608Metric, symbol Device:R_Small
- J1: footprint nrfmicro:USB-C_C168688 -> nrfmicro:HRO-TYPE-C-31-M-12
Connections:
- net P0.07: now also J6.3 (Pin_3)
- net P0.12: now also J6.4 (Pin_4)
- net P0.22: now also J5.4 (Pin_4)
- net P0.26: now also J6.2 (Pin_2)
- net P1.00: now also J5.3 (Pin_3)
- net P1.02: now also J5.2 (Pin_2)
- net P1.04: now also J5.1 (Pin_1)
- net at D3.1 (K): now also R8.1
- net at U3.1 (STAT): now also R8.2
- net BLUE_LED renamed P1.10
- net P1.10: now also J6.1 (Pin_1)
- no-connect marks 0 -> 1
